File: Lyra Avionics.kicad_sch (KiCad schematic)
At the start: 58 parts, among them SW1 SW_Push, SW2 SW_Push, U1 RP2350_80QFN, U2 LSM6DSV16XTR, U3 W25Q128JVS, U4 SMA-KWE_C20415790, U5 GT-USB-7010ASV, U6 RA-01SH, U7 NCP1117-3.3_SOT223, U8 BME280, U9 MPM3610AGQV-Z, Y1 ABM8-272-T3

Commit message: Completed first revision of PCB
Fully routed and checked in tolerance with JLCPCB manufacturing capabilities for 4L boards. Schematic needs checking and LCSC parts need assigning.
Parts:
- removed C26, C27: 22u, Capacitor_SMD:C_0805_2012Metric, symbol Device:C
- removed C28: 10u, Capacitor_SMD:C_0805_2012Metric, symbol Device:C
- removed R22: 24k, Resistor_SMD:R_0402_1005Metric, symbol Device:R
- removed U7: NCP1117-3.3_SOT223, Package_TO_SOT_SMD:SOT-223-3_TabPin2, symbol Regulator_Linear:NCP1117-3.3_SOT223
- removed U9: MPM3610AGQV-Z, footprint:QFN-20_L5.0-W3.0-P0.50-TL_MPM3610AGQV, symbol MPM3610AGQV-Z:MPM3610AGQV-Z
- added C1, C5: 100n, Capacitor_SMD:C_0402_1005Metric, symbol Device:C
- added C19, C22: 22u, Capacitor_SMD:C_0805_2012Metric, symbol Device:C
- added D1, D2: SS34, PCM_JLCPCB:D_SMA, symbol PCM_JLCPCB-Diodes:Schottky,SS34
- added L2: PA4332_222NLT, footprint:IND-SMD_L4.2-W4.2_PA4332, symbol PA4332_222NLT:PA4332_222NLT
- added R1: 10k, footprint:R0402, symbol 0402WGF1002TCE:0402WGF1002TCE
- added R11, R16, R17, R9: 4.7k, Resistor_SMD:R_0402_1005Metric, symbol Device:R
- added R13: 100k, Resistor_SMD:R_0402_1005Metric, symbol Device:R
- added U10, U9: QWIIC/Stemma I2C, footprint:CONN-SMD_4P-P1.00_SM04B-SRSS-TB-LF-SN, symbol SM04B-SRSS-TB_(LF)(SN):SM04B-SRSS-TB_(LF)(SN)
- added U7: TPS62162DSG, footprint:WSON-8_L2.0-W2.0-P0.50-TL-EP, symbol TPS62162DSG:TPS62162DSG
- R14, R15: value 75k -> 4.7k
Connections:
- net +3V3: now also R15.2, U2.5 (Vdd_IO), U2.8 (Vdd), C1.1, C19.1, C5.1, L2.2, R1.2, R11.2, R13.1, R16.2, R17.2, R9.2, U10.2, U7.6 (VOS), U9.2
- net GND: now also U2.6 (GND), U2.7 (GND), C1.2, C19.2, C22.2, C5.2, U10.1, U10.5, U10.6, U7.1 (PGND), U7.4 (AGND), U7.5 (FB), U7.9 (EP), U9.1, U9.5, U9.6
- net GPIO14: now also U6.6 (DIO1)
- net GPIO15: now also U6.4 (RESET)
- net GPIO16: now also U6.13 (MISO)
- net GPIO17: now also U6.15 (NSS)
- net GPIO18: now also U6.10 (BUSY)
- net GPIO19: now also U6.12 (SCK)
- net GPIO2: now also R14.1, R17.1, U10.3, U9.3
- net GPIO20: now also U6.14 (MOSI)
- net GPIO3: now also R15.1, R16.1, U10.4, U9.4
- net GPIO4: now also U2.14 (SDA), R9.1
- net GPIO5: now also U2.13 (SCL), R11.1
- net VBAT: now also D2.2; no longer R15.2
- net VBUS: now also D1.2
- net at U2.12 (CS): now also R1.1
- new net: R13.2, U7.8 (PG)
- new net: C22.1, D1.1, D2.1, U7.2 (VIN), U7.3 (EN)
- new net: L2.1, U7.7 (SW)
- no-connect marks 11 -> 13

Commit message: Added local library
Parts:
- C1, C10, C11, C12, C13, C14, C15, C16, C17, C18, C19, C2, C20, C21, C22, C24, C25, C3, C30, C31, C33, C4, C5, C6, C7, C8, C9: symbol Device:C -> Library:C
- D1, D2: symbol PCM_JLCPCB-Diodes:Schottky,SS34 -> Library:Schottky,SS34
- H1, H2, H3, H4: symbol Mechanical:MountingHole -> Library:MountingHole
- L1: symbol Device:L -> Library:L
- L2: symbol PA4332_222NLT:PA4332_222NLT -> Library:PA4332_222NLT
- R1: symbol 0402WGF1002TCE:0402WGF1002TCE -> Library:0402WGF1002TCE
- R10, R11, R13, R14, R15, R16, R17, R2, R24, R25, R26, R3, R4, R6, R7, R8, R9: symbol Device:R -> Library:R
- R12, R5: symbol PCM_SparkFun-Resistor:5.1k_0402 -> Library:5.1k_0402
- SW1, SW2: symbol Switch:SW_Push -> Library:SW_Push
- U1: symbol MCU_RaspberryPi_RP2350:RP2350_80QFN -> Library:RP2350_80QFN
- U10, U9: symbol SM04B-SRSS-TB_(LF)(SN):SM04B-SRSS-TB_(LF)(SN) -> Library:SM04B-SRSS-TB_(LF)(SN)
- U2: symbol LSM6DSV16XTR:LSM6DSV16XTR -> Library:LSM6DSV16XTR
- U3: symbol Memory_Flash:W25Q128JVS -> Library:W25Q128JVS
- U4: symbol SMA-KWE_C20415790:SMA-KWE_C20415790 -> Library:SMA-KWE_C20415790
- U5: symbol easyeda2kicad:GT-USB-7010ASV -> Library:GT-USB-7010ASV
- U6: symbol RA-01SH:RA-01SH -> Library:RA-01SH
- U7: symbol TPS62162DSG:TPS62162DSG -> Library:TPS62162DSG
- U8: symbol JLC2KICAD:BME280 -> Library:BME280
- Y1: symbol Device:Crystal_GND24 -> Library:Crystal_GND24

Commit message: Initial minor fixes of routing
Parts:
- added CN1: S2B-PH-SM4-TB(LF)(SN), Connectors:CONN-SMD_P2.00_S2B-PH-SM4-TB-LF-SN, symbol Connectors:S2B-PH-SM4-TB(LF)(SN)
Connections:
- net GND: now also CN1.2
- net VBAT: now also CN1.1
- no-connect marks 13 -> 15
