File: Lyra Avionics_2.kicad_sch (KiCad schematic)
At the start: 68 parts, among them SW1 SW_Push, SW2 SW_Push, U1 RP2350_80QFN, U10 QWIIC/Stemma I2C, U2 LSM6DSV16XTR, U3 W25Q128JVS, U4 SMA-KWE_C20415790, U5 GT-USB-7010ASV, U6 RA-01SH, U7 TPS62162DSG, U8 BME280, U9 QWIIC/Stemma I2C, Y1 ABM8-272-T3

Commit message: Fix
Parts:
- added CN1: S2B-PH-SM4-TB(LF)(SN), Connectors:CONN-SMD_P2.00_S2B-PH-SM4-TB-LF-SN, symbol Connectors:S2B-PH-SM4-TB(LF)(SN)
- C1, C10, C11, C12, C13, C14, C15, C16, C17, C18, C19, C2, C20, C21, C22, C24, C25, C3, C30, C31, C33, C4, C5, C6, C7, C8, C9: symbol Device:C -> Library:C
- D1, D2: symbol PCM_JLCPCB-Diodes:Schottky,SS34 -> Library:Schottky,SS34
- H1, H2, H3, H4: symbol Mechanical:MountingHole -> Library:MountingHole
- L1: symbol Device:L -> Library:L
- L2: symbol PA4332_222NLT:PA4332_222NLT -> Library:PA4332_222NLT
- R1: symbol 0402WGF1002TCE:0402WGF1002TCE -> Library:0402WGF1002TCE
- R10, R11, R13, R14, R15, R16, R17, R2, R24, R25, R26, R3, R4, R6, R7, R8, R9: symbol Device:R -> Library:R
- R12, R5: symbol PCM_SparkFun-Resistor:5.1k_0402 -> Library:5.1k_0402
- SW1, SW2: symbol Switch:SW_Push -> Library:SW_Push
- U1: symbol MCU_RaspberryPi_RP2350:RP2350_80QFN -> Library:RP2350_80QFN
- U10, U9: symbol SM04B-SRSS-TB_(LF)(SN):SM04B-SRSS-TB_(LF)(SN) -> Library:SM04B-SRSS-TB_(LF)(SN)
- U2: symbol LSM6DSV16XTR:LSM6DSV16XTR -> Library:LSM6DSV16XTR
- U3: symbol Memory_Flash:W25Q128JVS -> Library:W25Q128JVS
- U4: symbol SMA-KWE_C20415790:SMA-KWE_C20415790 -> Library:SMA-KWE_C20415790
- U5: symbol easyeda2kicad:GT-USB-7010ASV -> Library:GT-USB-7010ASV
- U6: symbol RA-01SH:RA-01SH -> Library:RA-01SH
- U7: symbol TPS62162DSG:TPS62162DSG -> Library:TPS62162DSG
- U8: symbol JLC2KICAD:BME280 -> Library:BME280
- Y1: symbol Device:Crystal_GND24 -> Library:Crystal_GND24
Connections:
- net +3V3: no longer U3.8 (VCC)
- net FLASH_SS: no longer U3.1 (~{CS})
- net GND: now also CN1.2; no longer U3.4 (GND)
- net QSPI_SCLK: no longer U3.6 (CLK)
- net QSPI_SD0: no longer U3.5 (DI(IO0))
- net QSPI_SD1: no longer U3.2 (DO(IO1))
- net QSPI_SD2: no longer U3.3 (IO2)
- net QSPI_SD3: no longer U3.7 (IO3)
- net VBAT: now also CN1.1
- no-connect marks 13 -> 15
Other:
- moved on the sheet: U3
